File: kit.kicad_sch (KiCad schematic)
At the start: 68 parts, among them IC1 TPA6130A2RTJR, J1 SJ-43617-SMT-TR, J2 Conn_01x06, U1 ESP32-S3-WROOM-1, U2 PCM5100A, U3 MIC5504-3.3YM5

Commit message: Updates
Parts:
- removed C11, C8: 0.47uF, Capacitor_SMD:C_01005_0402Metric, symbol Device:C_Small
- renumbered PLAY1 to ALT2
Connections:
- net LCM_DIN is gone; now on net PCM_DIN: U1.7 (IO7)
- net +3.3V: now also U2.1 (CPVDD)
- net SW_5: now also U1.31 (IO38); no longer U1.28 (IO35)
- net SW_6: now also U1.30 (IO37); no longer U1.29 (IO36)
- net SW_7: now also U1.29 (IO36); no longer U1.30 (IO37)
- net SW_8: now also U1.28 (IO35); no longer U1.31 (IO38)
- net SW_ALT: now also ALT2.1, ALT2.3; no longer PLAY1.1, PLAY1.3
- net SW_PLAY: now also PLAY1.1, PLAY1.3; no longer ALT2.1, ALT2.3
- net USB_DN: now also J2.4 (Pin_4); no longer J2.3 (Pin_3)
- net USB_DP: now also J2.3 (Pin_3); no longer J2.4 (Pin_4)
- net at C2.1, R10.2: now also IC1.5 (RIGHTINM)
- net at C3.2, R9.2: now also IC1.1 (LEFTINM)
Changed lines of the file:
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@@
 	)
 	(junction
+		(at 110.49 21.59)
+		(diameter 0)
+		(color 0 0 0 0)
+	)
+	(junction
 		(at 132.08 21.59)
 		(diameter 0)
@@
 	(wire
 		(pts
-			(xy 200.66 63.5) (xy 205.74 63.5)
+			(xy 200.66 63.5) (xy 214.63 63.5)
 		)
 		(stroke
@@
 	(wire
 		(pts
+			(xy 143.51 31.75) (xy 143.51 26.67)
+		)
+		(stroke
+			(width 0)
+			(type default)
+		)
+	)
+	(wire
+		(pts
 			(xy -10.16 99.06) (xy 10.16 99.06)
 		)
@@
 	(wire
 		(pts
+			(xy 110.49 26.67) (xy 110.49 21.59)
+		)
+		(stroke
+			(width 0)
+			(type default)
+		)
+	)
+	(wire
+		(pts
 			(xy 171.45 36.83) (xy 184.15 36.83)
 		)
@@
 	(wire
 		(pts
+			(xy 143.51 26.67) (xy 110.49 26.67)
+		)
+		(stroke
+			(width 0)
+			(type default)
+		)
+	)
+	(wire
+		(pts
 			(xy 267.97 45.72) (xy 267.97 85.09)
 		)
@@
 	(wire
 		(pts
-			(xy 201.93 33.02) (xy 205.74 33.02)
+			(xy 201.93 33.02) (xy 223.52 33.02)
 		)
 		(stroke
@@
 	(wire
 		(pts
-			(xy 214.63 63.5) (xy 210.82 63.5)
-		)
-		(stroke
-			(width 0)
-			(type default)
-		)
-	)
-	(wire
-		(pts
 			(xy 8.89 231.14) (xy 8.89 224.79)
 		)
@@
 	(wire
 		(pts
-			(xy 210.82 33.02) (xy 223.52 33.02)
-		)
-		(stroke
-			(width 0)
-			(type default)
-		)
-	)
-	(wire
-		(pts
 			(xy 64.77 39.37) (xy 60.96 39.37)
 		)
@@
 	)
 	(label "USB_DP"
-		(at 101.6 138.43 180)
+		(at 101.6 135.89 180)
 		(effects
 			(font
@@
 	)
 	(label "SW_8"
-		(at 99.06 81.28 0)
+		(at 99.06 73.66 0)
 		(effects
 			(font
@@
 	)
 	(label "SW_7"
-		(at 99.06 78.74 0)
+		(at 99.06 76.2 0)
 		(effects
 			(font
@@
 	)
 	(label "SW_ALT"
-		(at 10.16 205.74 0)
+		(at 8.89 222.25 0)
 		(effects
 			(font
@@
 		)
 	)
-	(label "LCM_DIN"
+	(label "PCM_DIN"
 		(at 68.58 78.74 180)
 		(effects
@@
 	)
 	(label "SW_6"
-		(at 99.06 76.2 0)
+		(at 99.06 78.74 0)
 		(effects
 			(font
@@
 	)
 	(label "USB_DN"
-		(at 101.6 135.89 180)
+		(at 101.6 138.43 180)
 		(effects
 			(font
@@
 	)
 	(label "SW_5"
-		(at 99.06 73.66 0)
+		(at 99.06 81.28 0)
 		(effects
 			(font
@@
 	)
 	(label "SW_PLAY"
-		(at 8.89 222.25 0)
+		(at 10.16 205.74 0)
 		(effects
 			(font
@@
 		(dnp no)
 		(fields_autoplaced yes)
-		(property "Reference" "PLAY1"
+		(property "Reference" "ALT2"
 			(at -1.27 214.63 0)
 			(effects
@@
 			(project "kit"
 				(path "/63a38faa-4ddd-4745-8fe9-8662e2dcf4e4"
-					(reference "PLAY1")
-					(unit 1)
-				)
-			)
-		)
-	)
-	(symbol
-		(lib_id "Device:C_Small")
-		(at 208.28 33.02 90)
-		(unit 1)
-		(exclude_from_sim no)
-		(in_bom yes)
-		(on_board yes)
-		(dnp no)
-		(fields_autoplaced yes)
-		(property "Reference" "C8"
-			(at 208.2863 26.67 90)
-			(effects
-				(font
-					(size 1.27 1.27)
-				)
-			)
-		)
-		(property "Value" "0.47uF"
-			(at 208.2863 29.21 90)
-			(effects
-				(font
-					(size 1.27 1.27)
-				)
-			)
-		)
-		(property "Footprint" "Capacitor_SMD:C_01005_0402Metric"
-			(at 208.28 33.02 0)
-			(effects
-				(font
-					(size 1.27 1.27)
-				)
-				(hide yes)
-			)
-		)
-		(property "Datasheet" "~"
-			(at 208.28 33.02 0)
-			(effects
-				(font
-					(size 1.27 1.27)
-				)
-				(hide yes)
-			)
-		)
-		(property "Description" "Unpolarized capacitor, small symbol"
-			(at 208.28 33.02 0)
-			(effects
-				(font
-					(size 1.27 1.27)
-				)
-				(hide yes)
-			)
-		)
-		(pin "1"
-		)
-		(pin "2"
-		)
-		(instances
-			(project ""
-				(path "/63a38faa-4ddd-4745-8fe9-8662e2dcf4e4"
-					(reference "C8")
+					(reference "ALT2")
 					(unit 1)
 				)
@@
 					(unit 1)
 				)
-			)
-		)
-	)
-	(symbol
-		(lib_id "Device:C_Small")
-		(at 208.28 63.5 90)
-		(unit 1)
-		(exclude_from_sim no)
-		(in_bom yes)
-		(on_board yes)
-		(dnp no)
-		(fields_autoplaced yes)
-		(property "Reference" "C11"
-			(at 208.2863 57.15 90)
-			(effects
-				(font
-					(size 1.27 1.27)
-				)
-			)
-		)
-		(property "Value" "0.47uF"
-			(at 208.2863 59.69 90)
-			(effects
-				(font
-					(size 1.27 1.27)
-				)
-			)
-		)
-		(property "Footprint" "Capacitor_SMD:C_01005_0402Metric"
-			(at 208.28 63.5 0)
-			(effects
-				(font
-					(size 1.27 1.27)
-				)
-				(hide yes)
-			)
-		)
-		(property "Datasheet" "~"
-			(at 208.28 63.5 0)
-			(effects
-				(font
-					(size 1.27 1.27)
-				)
-				(hide yes)
-			)
-		)
-		(property "Description" "Unpolarized capacitor, small symbol"
-			(at 208.28 63.5 0)
-			(effects
-				(font
-					(size 1.27 1.27)
-				)
-				(hide yes)
-			)
-		)
-		(pin "1"
-		)
-		(pin "2"
-		)
-		(instances
-			(project ""
-				(path "/63a38faa-4ddd-4745-8fe9-8662e2dcf4e4"
-					(reference "C11")
-					(unit 1)
-				)
